Commit message: chore: follow the description package rename to litearm_description
The arm's description package is `litearm_description` now (was `litearm_urdf`;
the repository was renamed litearm-urdf -> litearm-description). This application
bundles its own copy of the model, so nothing was broken, but the bundled
package name was still the old one:

- `public/description/litearm.urdf`: the robot name and the 18
  `package://` mesh URIs
- `src/components/RobotViewport.tsx`: the URDFLoader `packages` key, which has to
  match those URIs

The bundled file name (`litearm.urdf`) and the mesh files are unchanged.

File: public/description/litearm.urdf (robot description, URDF)
Before this commit: robot litearm_urdf, 9 links, 8 joints
Links:
- link Link1: geometry collision mesh filename=package://litearm_description/meshes/Link1.STL; visual mesh filename=package://litearm_description/meshes/Link1.STL
- link Link2: geometry collision mesh filename=package://litearm_description/meshes/Link2.STL; visual mesh filename=package://litearm_description/meshes/Link2.STL
- link Link3: geometry collision mesh filename=package://litearm_description/meshes/Link3.STL; visual mesh filename=package://litearm_description/meshes/Link3.STL
- link Link4: geometry collision mesh filename=package://litearm_description/meshes/Link4.STL; visual mesh filename=package://litearm_description/meshes/Link4.STL
- link Link5: geometry collision mesh filename=package://litearm_description/meshes/Link5.STL; visual mesh filename=package://litearm_description/meshes/Link5.STL
- link Link6: geometry collision mesh filename=package://litearm_description/meshes/Link6.STL; visual mesh filename=package://litearm_description/meshes/Link6.STL
- link Link7: geometry collision mesh filename=package://litearm_description/meshes/Link7.STL; visual mesh filename=package://litearm_description/meshes/Link7.STL
- link base_link: geometry collision mesh filename=package://litearm_description/meshes/base_link.STL; visual mesh filename=package://litearm_description/meshes/base_link.STL
- link ee_frame_link: geometry collision mesh filename=package://litearm_description/meshes/ee_frame_link.STL; visual mesh filename=package://litearm_description/meshes/ee_frame_link.STL
